File: VolOsc.kicad_sch (KiCad schematic)
At the start: 27 parts, among them Q10 SMP5484, Q11 MMBT3906, Q12 MMBT3906

Commit message: Components mostly placed
Parts:
- C30, C31: footprint Capacitor_Tantalum_SMD:CP_EIA-1608-08_AVX-J -> Capacitor_Tantalum_SMD:CP_EIA-2012-12_Kemet-R_Pad1.30x1.05mm_HandSolder
Changed lines of the file:
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@@
       (effects (font (size 1.27 1.27)) (justify left))
     )
-    (property "Footprint" "Capacitor_Tantalum_SMD:CP_EIA-1608-08_AVX-J" (id 2) (at 107.95 132.715 0)
+    (property "Footprint" "Capacitor_Tantalum_SMD:CP_EIA-2012-12_Kemet-R_Pad1.30x1.05mm_HandSolder" (id 2) (at 107.95 132.715 0)
       (effects (font (size 1.27 1.27)) hide)
     )
@@
       (effects (font (size 1.27 1.27)) (justify left))
     )
-    (property "Footprint" "Capacitor_Tantalum_SMD:CP_EIA-1608-08_AVX-J" (id 2) (at 149.225 89.535 0)
-      (effects (font (size 1.27 1.27)) hide)
-    )
+    (property "Footprint" "Capacitor_Tantalum_SMD:CP_EIA-2012-12_Kemet-R_Pad1.30x1.05mm_HandSolder" (id 2) (at 149.225 89.535 0)
+      (effects (font (size 1.27 1.27)) hide)
+    )

Commit message: Better component placements
Parts:
- added JP4: D, Jumper:SolderJumper-2_P1.3mm_Open_RoundedPad1.0x1.5mm, symbol Jumper:SolderJumper_2_Open
- added TP4: TestPoint, TestPoint:TestPoint_Loop_D1.80mm_Drill1.0mm_Beaded, symbol Connector:TestPoint
- TP1, TP2, TP3: footprint TestPoint:TestPoint_Pad_D1.0mm -> TestPoint:TestPoint_Loop_D1.80mm_Drill1.0mm_Beaded
Connections:
- net D: now also JP4.2 (B); no longer Q10.1 (S), R31.1
- new net: JP4.1 (A), Q10.1 (S), R31.1, TP4.1
Other:
- moved on the sheet: C25, C26, C27, C28, C29, C30, C31, CR4, CR5, L4, Q10, Q11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
