File: pitch_osc.kicad_sch (KiCad schematic)
At the start: 29 parts, among them Q1 MMBT3906, Q2 MMBT3906, Q3 SMP5484

Commit message: Components mostly placed
Parts:
- C1, C2: footprint Capacitor_Tantalum_SMD:CP_EIA-1608-08_AVX-J -> Capacitor_Tantalum_SMD:CP_EIA-2012-12_Kemet-R_Pad1.30x1.05mm_HandSolder
- C6: footprint Theremin:CAPV_JZ400 -> Capacitor_SMD:C_1210_3225Metric_Pad1.33x2.70mm_HandSolder
- C7: footprint Inductor_SMD:L_0805_2012Metric_Pad1.05x1.20mm_HandSolder -> Theremin:CAPV_JZ400
Changed lines of the file:
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@@
       (effects (font (size 1.27 1.27)) (justify left))
     )
-    (property "Footprint" "Capacitor_Tantalum_SMD:CP_EIA-1608-08_AVX-J" (id 2) (at 106.68 54.61 0)
+    (property "Footprint" "Capacitor_Tantalum_SMD:CP_EIA-2012-12_Kemet-R_Pad1.30x1.05mm_HandSolder" (id 2) (at 106.68 54.61 0)
       (effects (font (size 1.27 1.27)) hide)
     )
@@
       (effects (font (size 1.27 1.27)) (justify left))
     )
-    (property "Footprint" "Theremin:CAPV_JZ400" (id 2) (at 116.5352 97.155 0)
+    (property "Footprint" "Capacitor_SMD:C_1210_3225Metric_Pad1.33x2.70mm_HandSolder" (id 2) (at 116.5352 97.155 0)
       (effects (font (size 1.27 1.27)) hide)
     )
@@
       (effects (font (size 1.27 1.27)) (justify left))
     )
-    (property "Footprint" "Capacitor_Tantalum_SMD:CP_EIA-1608-08_AVX-J" (id 2) (at 65.405 97.79 0)
+    (property "Footprint" "Capacitor_Tantalum_SMD:CP_EIA-2012-12_Kemet-R_Pad1.30x1.05mm_HandSolder" (id 2) (at 65.405 97.79 0)
       (effects (font (size 1.27 1.27)) hide)
     )
@@
       (effects (font (size 1.27 1.27)) (justify left))
     )
-    (property "Footprint" "Inductor_SMD:L_0805_2012Metric_Pad1.05x1.20mm_HandSolder" (id 2) (at 129.54 93.345 0)
-      (effects (font (size 1.27 1.27)) hide)
-    )
+    (property "Footprint" "Theremin:CAPV_JZ400" (id 2) (at 129.54 93.345 0)
+      (effects (font (size 1.27 1.27)) hide)
+    )

Commit message: Better component placements
Parts:
- removed TP10, TP9: TestPoint, TestPoint:TestPoint_Pad_D1.0mm, symbol Connector:TestPoint
- added JP6: F, Jumper:SolderJumper-2_P1.3mm_Open_RoundedPad1.0x1.5mm, symbol Jumper:SolderJumper_2_Open
- TP8: footprint TestPoint:TestPoint_Pad_D1.0mm -> TestPoint:TestPoint_Loop_D1.80mm_Drill1.0mm_Beaded
Connections:
- net F: now also JP6.2 (B); no longer C8.2
- new net: C8.2, JP6.1 (A)
Changed lines of the file:
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@@
   (junction (at 161.29 84.455) (diameter 0) (color 0 0 0 0)
   )
-  (junction (at 57.785 100.33) (diameter 0) (color 0 0 0 0)
-  )
   (junction (at 78.105 93.345) (diameter 0) (color 0 0 0 0)
   )
@@
     (stroke (width 0) (type default) (color 0 0 0 0))
   )
-  (wire (pts (xy 57.785 100.33) (xy 54.61 100.33))
-    (stroke (width 0) (type default) (color 0 0 0 0))
-  )
   (wire (pts (xy 57.785 101.6) (xy 65.405 101.6))
     (stroke (width 0) (type default) (color 0 0 0 0))
@@
     (stroke (width 0) (type default) (color 0 0 0 0))
   )
-  (wire (pts (xy 57.785 100.33) (xy 57.785 101.6))
-    (stroke (width 0) (type default) (color 0 0 0 0))
-  )
   (wire (pts (xy 65.405 100.33) (xy 65.405 101.6))
     (stroke (width 0) (type default) (color 0 0 0 0))
@@
     (stroke (width 0) (type default) (color 0 0 0 0))
   )
+  (wire (pts (xy 166.37 55.88) (xy 176.53 55.88))
+    (stroke (width 0) (type default) (color 0 0 0 0))
+  )
   (wire (pts (xy 91.44 36.83) (xy 143.51 36.83))
     (stroke (width 0) (type default) (color 0 0 0 0))
@@
     (stroke (width 0) (type default) (color 0 0 0 0))
   )
-  (wire (pts (xy 166.37 55.88) (xy 177.8 55.88))
-    (stroke (width 0) (type default) (color 0 0 0 0))
-  )
-  (wire (pts (xy 65.405 89.535) (xy 65.405 93.345))
-    (stroke (width 0) (type default) (color 0 0 0 0))
-  )
   (wire (pts (xy 115.57 76.2) (xy 115.57 84.455))
     (stroke (width 0) (type default) (color 0 0 0 0))
@@
     (stroke (width 0) (type default) (color 0 0 0 0))
   )
+  (wire (pts (xy 184.15 55.88) (xy 193.04 55.88))
+    (stroke (width 0) (type default) (color 0 0 0 0))
+  )
   (wire (pts (xy 95.25 57.15) (xy 95.25 62.23))
     (stroke (width 0) (type default) (color 0 0 0 0))
@@
     (stroke (width 0) (type default) (color 0 0 0 0))
   )
-  (wire (pts (xy 57.785 97.155) (xy 57.785 100.33))
+  (wire (pts (xy 57.785 97.155) (xy 57.785 101.6))
     (stroke (width 0) (type default) (color 0 0 0 0))
   )
@@
     )
   )
-  (global_label "F" (shape input) (at 177.8 55.88 0) (fields_autoplaced)
+  (global_label "F" (shape input) (at 193.04 55.88 0) (fields_autoplaced)
     (effects (font (size 1.27 1.27)) (justify left))
-    (property "Intersheet References" "${INTERSHEET_REFS}" (id 0) (at 181.3017 55.8006 0)
+    (property "Intersheet References" "${INTERSHEET_REFS}" (id 0) (at 196.5417 55.8006 0)
       (effects (font (size 1.27 1.27)) (justify left) hide)
     )
@@
       (effects (font (size 1.27 1.27)) (justify left) hide)
     )
-    (property "Footprint" "TestPoint:TestPoint_Pad_D1.0mm" (id 2) (at 54.61 80.01 0)
+    (property "Footprint" "TestPoint:TestPoint_Loop_D1.80mm_Drill1.0mm_Beaded" (id 2) (at 54.61 80.01 0)
       (effects (font (size 1.27 1.27)) hide)
     )
     (property "Datasheet" "~" (id 3) (at 54.61 80.01 0)
-      (effects (font (size 1.27 1.27)) hide)
-    )
-    (pin "1")
-  )
-  (symbol (lib_id "Connector:TestPoint") (at 65.405 89.535 0) (unit 1)
-    (in_bom yes) (on_board yes)
-    (property "Reference" "TP9" (id 0) (at 63.5 83.82 0)
-      (effects (font (size 1.27 1.27)) (justify left))
-    )
-    (property "Value" "TestPoint" (id 1) (at 67.31 87.5029 0)
-      (effects (font (size 1.27 1.27)) (justify left) hide)
-    )
-    (property "Footprint" "TestPoint:TestPoint_Pad_D1.0mm" (id 2) (at 70.485 89.535 0)
-      (effects (font (size 1.27 1.27)) hide)
-    )
-    (property "Datasheet" "~" (id 3) (at 70.485 89.535 0)
       (effects (font (size 1.27 1.27)) hide)
     )
@@
     (pin "1")
     (pin "2")
-  )
-  (symbol (lib_id "Connector:TestPoint") (at 54.61 100.33 90) (unit 1)
-    (in_bom yes) (on_board yes)
-    (property "Reference" "TP10" (id 0) (at 48.895 102.235 0)
-      (effects (font (size 1.27 1.27)) (justify left))
-    )
-    (property "Value" "TestPoint" (id 1) (at 52.5779 98.425 0)
-      (effects (font (size 1.27 1.27)) (justify left) hide)
-    )
-    (property "Footprint" "TestPoint:TestPoint_Pad_D1.0mm" (id 2) (at 54.61 95.25 0)
-      (effects (font (size 1.27 1.27)) hide)
-    )
-    (property "Datasheet" "~" (id 3) (at 54.61 95.25 0)
-      (effects (font (size 1.27 1.27)) hide)
-    )
-    (pin "1")
   )
   (symbol (lib_id "Device:R_Small_US") (at 71.755 93.345 90) (unit 1)
@@
       (effects (font (size 1.27 1.27)) hide)
     )
+    (pin "1")
+    (pin "2")
+  )
+  (symbol (lib_id "Jumper:SolderJumper_2_Open") (at 180.34 55.88 0) (unit 1)
+    (in_bom yes) (on_board yes) (fields_autoplaced)
+    (property "Reference" "JP6" (id 0) (at 180.34 49.53 0))
+    (property "Value" "F" (id 1) (at 180.34 52.07 0))
+    (property "Footprint" "Jumper:SolderJumper-2_P1.3mm_Open_RoundedPad1.0x1.5mm" (id 2) (at 180.34 55.88 0)
+      (effects (font (size 1.27 1.27)) hide)
+    )
+    (property "Datasheet" "~" (id 3) (at 180.34 55.88 0)
+      (effects (font (size 1.27 1.27)) hide)
+    )
