File: AudioAmpVreg.kicad_sch (KiCad schematic)
At the start: 40 parts, among them J3 M3_PTH, J4 M3_PTH, Q14 MMBT3904, Q15 MMBT3904, Q16 MMBT3906, SW1 SW_SPDT, U1 LDK320-ADJ_SOT23_SOT353

Commit message: Components mostly placed
Parts:
- removed BT1: +9V, Battery:BatteryHolder_Eagle_12BH611-GR, symbol Device:Battery_Cell
- removed SW1: SW_SPDT, Theremin:CSS1210TB, symbol Switch:SW_SPDT
- removed TP12, TP13, TP6, TP7: TestPoint, TestPoint:TestPoint_Pad_D1.0mm, symbol Connector:TestPoint
- added J5: 9V IN, MountingHole:MountingHole_4.3mm_M4_Pad_Via, symbol Connector_Generic:Conn_01x01
- C33, C41: footprint Capacitor_Tantalum_SMD:CP_EIA-1608-08_AVX-J -> Capacitor_Tantalum_SMD:CP_EIA-2012-12_Kemet-R_Pad1.30x1.05mm_HandSolder
- D1: footprint LED_SMD:LED_0201_0603Metric -> LED_SMD:LED_0603_1608Metric_Pad1.05x0.95mm_HandSolder
- J3: value M3_PTH -> GROUND POINT; footprint MountingHole:MountingHole_3.2mm_M3_Pad_Via -> MountingHole:MountingHole_4.3mm_M4_Pad_Via
- J4: value M3_PTH -> LINE OUT; footprint MountingHole:MountingHole_3.2mm_M3_Pad_Via -> MountingHole:MountingHole_4.3mm_M4_Pad_Via
Connections:
- net +9V: now also J5.1 (Pin_1)
- no-connect marks 1 -> 0
Other:
- moved on the sheet: C32, C33, C41, CR6, D1, J3, R56, R57, R58, U1

Commit message: Better component placements
Parts:
- added JP5: E, Jumper:SolderJumper-2_P1.3mm_Open_RoundedPad1.0x1.5mm, symbol Jumper:SolderJumper_2_Open
- added TP7: TestPoint, TestPoint:TestPoint_Loop_D1.80mm_Drill1.0mm_Beaded, symbol Connector:TestPoint
- TP5: footprint TestPoint:TestPoint_Pad_D1.0mm -> TestPoint:TestPoint_Loop_D1.80mm_Drill1.0mm_Beaded
Connections:
- net E: now also JP5.1 (A); no longer C35.1
- net at C36.1, C38.1, Q14.3 (C)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: now also TP7.1
- new net: C35.1, JP5.2 (B)
Changed lines of the file:
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@@
   (junction (at 198.12 62.23) (diameter 0) (color 0 0 0 0)
   )
+  (junction (at 115.57 109.22) (diameter 0) (color 0 0 0 0)
+  )
   (junction (at 198.12 39.37) (diameter 0) (color 0 0 0 0)
   )
@@
     (stroke (width 0) (type default) (color 0 0 0 0))
   )
+  (wire (pts (xy 59.69 116.84) (xy 63.5 116.84))
+    (stroke (width 0) (type default) (color 0 0 0 0))
+  )
   (wire (pts (xy 162.56 119.38) (xy 162.56 121.92))
     (stroke (width 0) (type default) (color 0 0 0 0))
@@
     (stroke (width 0) (type default) (color 0 0 0 0))
   )
+  (wire (pts (xy 115.57 104.14) (xy 115.57 109.22))
+    (stroke (width 0) (type default) (color 0 0 0 0))
+  )
   (wire (pts (xy 82.55 116.84) (xy 88.9 116.84))
     (stroke (width 0) (type default) (color 0 0 0 0))
@@
     (stroke (width 0) (type default) (color 0 0 0 0))
   )
-  (wire (pts (xy 59.69 116.84) (xy 73.66 116.84))
-    (stroke (width 0) (type default) (color 0 0 0 0))
-  )
   (wire (pts (xy 148.59 133.35) (xy 148.59 135.89))
     (stroke (width 0) (type default) (color 0 0 0 0))
@@
   )
   (wire (pts (xy 162.56 93.98) (xy 162.56 100.33))
+    (stroke (width 0) (type default) (color 0 0 0 0))
+  )
+  (wire (pts (xy 71.12 116.84) (xy 73.66 116.84))
     (stroke (width 0) (type default) (color 0 0 0 0))
   )
@@
     (pin "2")
   )
+  (symbol (lib_id "Connector:TestPoint") (at 115.57 104.14 0) (unit 1)
+    (in_bom yes) (on_board yes)
+    (property "Reference" "TP7" (id 0) (at 113.03 102.87 90)
+      (effects (font (size 1.27 1.27)) (justify left))
+    )
+    (property "Value" "TestPoint" (id 1) (at 117.475 102.1079 0)
+      (effects (font (size 1.27 1.27)) (justify left) hide)
+    )
+    (property "Footprint" "TestPoint:TestPoint_Loop_D1.80mm_Drill1.0mm_Beaded" (id 2) (at 120.65 104.14 0)
+      (effects (font (size 1.27 1.27)) hide)
+    )
+    (property "Datasheet" "~" (id 3) (at 120.65 104.14 0)
+      (effects (font (size 1.27 1.27)) hide)
+    )
+    (pin "1")
+  )
   (symbol (lib_id "Transistor_BJT:MMBT3904") (at 95.25 116.84 0) (unit 1)
     (in_bom yes) (on_board yes) (fields_autoplaced)
@@
     (pin "2")
   )
+  (symbol (lib_id "Jumper:SolderJumper_2_Open") (at 67.31 116.84 0) (unit 1)
+    (in_bom yes) (on_board yes) (fields_autoplaced)
+    (property "Reference" "JP5" (id 0) (at 67.31 110.49 0))
+    (property "Value" "E" (id 1) (at 67.31 113.03 0))
+    (property "Footprint" "Jumper:SolderJumper-2_P1.3mm_Open_RoundedPad1.0x1.5mm" (id 2) (at 67.31 116.84 0)
+      (effects (font (size 1.27 1.27)) hide)
+    )
+    (property "Datasheet" "~" (id 3) (at 67.31 116.84 0)
+      (effects (font (size 1.27 1.27)) hide)
+    )
+    (pin "1")
+    (pin "2")
+  )
   (symbol (lib_id "Transistor_BJT:MMBT3904") (at 160.02 105.41 0) (unit 1)
     (in_bom yes) (on_board yes) (fields_autoplaced)
@@
       (effects (font (size 1.27 1.27)) (justify left) hide)
     )
-    (property "Footprint" "TestPoint:TestPoint_Pad_D1.0mm" (id 2) (at 191.77 137.16 0)
-      (effects (font (size 1.27 1.27)) hide)
-    )
+    (property "Footprint" "TestPoint:TestPoint_Loop_D1.80mm_Drill1.0mm_Beaded" (id 2) (at 191.77 137.16 0)
+      (effects (font (size 1.27 1.27)) hide)
+    )

Commit message: Routing finished, still needs to pass DRC
Connections:
- net +7.5V: now also R43.2; no longer R43.1
- net at C36.1, C38.1, Q14.3 (C)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: now also R43.1; no longer R43.2
Other:
- moved on the sheet: R43
Changed lines of the file:
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@@
     (pin "2")
   )
-  (symbol (lib_id "Device:R_Small_US") (at 97.79 104.14 0) (unit 1)
+  (symbol (lib_id "Device:R_Small_US") (at 97.79 104.14 180) (unit 1)
     (in_bom yes) (on_board yes) (fields_autoplaced)
     (property "Reference" "R43" (id 0) (at 100.33 102.8699 0)
-      (effects (font (size 1.27 1.27)) (justify left))
+      (effects (font (size 1.27 1.27)) (justify right))
     )
     (property "Value" "680" (id 1) (at 100.33 105.4099 0)
-      (effects (font (size 1.27 1.27)) (justify left))
+      (effects (font (size 1.27 1.27)) (justify right))
     )
     (property "Footprint" "Resistor_SMD:R_0603_1608Metric" (id 2) (at 97.79 104.14 0)
