File: Harrison145.kicad_pcb (KiCad board)
At the start: 2 copper layers, 85 x 55 mm, 152 parts, among them J1 PITCH ANTENNA, J2 VOLUME ANTENNA, J3 GROUND POINT, J4 LINE OUT, J5 9V IN, Q1 MMBT3906, Q10 SMP5484, Q11 MMBT3906, Q12 MMBT3906, Q13 SMP5484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

Commit message: All DRC/ERC that matters passes
Parts:
- added G***: LOGO, Theremin:walrus, B.Cu at (160.5, 50.1)
- moved Ge 0.10 mm to (183.0, 79.4)
- turned R43 to 0 degrees
- renumbered G*** to Ge
Connections:
- R43 pad 1: +7.5V -> Net-(C36-Pad1)
- R43 pad 2: Net-(C36-Pad1) -> +7.5V
Routing:
- net Net-(C37-Pad2): track 5.33 -> 4.50 mm
Other:
- board text removed: "AMP"
- board text removed: "FPO"
- board text removed: "TODO: Make sure tantalum capacitors have directional indicators Buy test points and standoffs Resize silk text for all passives Scoot volume knob away from edge Hook test points for everything specified as needing scope connections Make sure layout still makes sense with double plate configuration Make sure all named test points are exposed and labeled Generate annotated BOM and attach datasheets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"
- board text removed: "VPO"
- board text removed: "VVO"

Commit message: Added revision number
Other:
- board text added: "12/13/2022 Rev 1"
Changed lines of the file:
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@@
   (gr_arc locked (start 140.5 60) (mid 142.843146 54.343146) (end 148.5 52) (layer "Edge.Cuts") (width 0.4))
   (gr_line locked (start 148.5 52) (end 217.5 52) (layer "Edge.Cuts") (width 0.4))
+  (gr_text "12/13/2022\nRev 1\n" (at 205.1 55.8) (layer "F.Cu")
+    (effects (font (size 0.8 0.8) (thickness 0.2)) (justify right))
+  )
+  (gr_text "12/13/2022\nRev 1\n" (at 205.1 55.8) (layer "F.Mask")
+    (effects (font (size 0.8 0.8) (thickness 0.2)) (justify right))
+  )
   (gr_text "FVO" (at 181.66 87.859998) (layer "Cmts.User")
     (effects (font (size 1.2 1.2) (thickness 0.2)))
