File: VarOsc.kicad_sch (KiCad schematic)
At the start: 18 parts, among them J1 PITCH ANTENNA, Q5 SMP5484, Q6 MMBT3906, Q7 MMBT3906

Commit message: Added iBOM
Parts:
- C14, C14_TEST1: DNP (none) -> 1
Changed lines of the file:
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@@
+      (effects (font (size 1.27 1.27)) hide)
+    )
+    (property "DNP" "1" (id 4) (at 143.51 100.33 0)
       (effects (font (size 1.27 1.27)) hide)
     )
@@
       (effects (font (size 1.27 1.27)) hide)
     )
+    (property "DNP" "1" (id 4) (at 184.15 100.33 0)
+      (effects (font (size 1.27 1.27)) hide)
+    )
