File: VolProcessor.kicad_sch (KiCad schematic)
At the start: 21 parts, among them J2 VOLUME ANTENNA, Q13 SMP5484, Q8 SMP5484, Q9 MMBT3904

Commit message: Added iBOM
Parts:
- C24, C24_TEST1: DNP (none) -> 1
Changed lines of the file:
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@@
+      (effects (font (size 1.27 1.27)) hide)
+    )
+    (property "DNP" "1" (id 4) (at 63.5 109.22 0)
       (effects (font (size 1.27 1.27)) hide)
     )
@@
       (effects (font (size 1.27 1.27)) hide)
     )
-    (pin "1")
-    (pin "2")
+    (property "DNP" "1" (id 4) (at 105.41 109.22 0))
+    (pin "1")
+    (pin "2")
