File: Harrison145_Main_Rev2/Harrison145.kicad_pcb (KiCad board)
At the start: 2 copper layers, 85 x 55 mm, 154 parts, among them J1 PITCH ANTENNA, J2 VOLUME ANTENNA, J3 GROUND POINT, J4 LINE OUT, J5 9V IN, Q1 MMBT3906, Q10 SMP5484, Q11 MMBT3906, Q12 MMBT3906, Q13 SMP5484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

Commit message: Update rev2 kicad_pcb
Parts:
- moved TP1 12.4 mm to (161.1, 89.3)
- moved TP2 6.04 mm to (170.2, 79.0)
- moved R6 4.30 mm to (165.2, 89.8), turned to -90 degrees
- moved C7 3.80 mm to (160.4, 93.3)
- moved R7 3.40 mm to (158.3, 89.8), turned to -90 degrees
- moved C6 3.36 mm to (160.2, 96.8)
- moved TP3 3.11 mm to (164.0, 69.8)
- moved R19 3.04 mm to (164.5, 67.0)
- moved R17 1.85 mm to (166.7, 78.5)
- moved R16 1.82 mm to (163.6, 78.5)
- moved R21 1.80 mm to (159.5, 66.0)
- moved C15 1.75 mm to (159.5, 64.2)
- moved CR1 1.68 mm to (156.0, 98.0)
- moved C13 1.47 mm to (173.0, 77.4), turned to -90 degrees
- moved R5 1.46 mm to (163.7, 86.8)
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Routing:
- net GND: track 457.0 -> 421.0 mm, vias 10 -> 9
- net C: track 25.1 -> 0.00 mm, vias 2 -> 0
- net Net-(Q14-C): track 28.0 -> 21.6 mm
- net Net-(J1-Pin_1): track 53.8 -> 47.8 mm
- net Net-(C39-Pad1): track 4.17 -> 0.00 mm
- net Net-(JP2-A): track 17.6 -> 21.3 mm
- net A: track 22.3 -> 19.0 mm
- net Net-(JP3-A): track 11.3 -> 8.56 mm
- net Net-(Q4-C): track 4.42 -> 6.16 mm
- net B: track 8.63 -> 7.00 mm
- net Net-(CR1-A): track 9.90 -> 11.5 mm
- net Net-(Q4-E): track 5.00 -> 3.44 mm
- net +7.5V: track 171.1 -> 172.6 mm
- net F: track 23.3 -> 21.9 mm
- net Net-(CR1-K): track 6.07 -> 4.73 mm
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
Commit message: Small updates
* Edited Errata
* Changed VReg resistor from 20k to 20.5k
* Changed ceramic cap symbols incorrectly listed as polarized
Parts:
- R56: value 20.0K -> 20.5K
Changed lines of the file:
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@@
         (effects (font (size 1 1) (thickness 0.15)))
     )
-    (fp_text value "20.0K" (at 0 1.43) (layer "F.Fab") hide
+    (fp_text value "20.5K" (at 0 1.43) (layer "F.Fab") hide
         (effects (font (size 1 1) (thickness 0.15)))
     )
@@
     (property "Sheetfile" "pitch_osc.kicad_sch")
     (property "Sheetname" "Pitch Reference Oscillator")
-    (property "ki_description" "Polarized capacitor, small US symbol")
-    (property "ki_keywords" "cap capacitor")
+    (property "ki_description" "Unpolarized capacitor, small symbol")
+    (property "ki_keywords" "capacitor cap")
     (attr smd)
     (fp_text reference "C3" (at 0 -1.43) (layer "F.SilkS") hide
@@
     (property "Sheetfile" "VolOsc.kicad_sch")
     (property "Sheetname" "Volume Oscillator")
-    (property "ki_description" "Polarized capacitor, small US symbol")
-    (property "ki_keywords" "cap capacitor")
+    (property "ki_description" "Unpolarized capacitor, small symbol")
+    (property "ki_keywords" "capacitor cap")
     (attr smd)
     (fp_text reference "C29" (at 0 -1.43 90) (layer "F.SilkS") hide
