File: Harrison145_Main_Rev2/AudioAmpVreg.kicad_sch (KiCad schematic)
At the start: 36 parts, among them J3 GROUND POINT, J4 LINE OUT, J5 9V IN, Q14 MMBT3904, Q15 MMBT3904, Q16 MMBT3906, U1 LDK320-ADJ_SOT23_SOT353

Commit message: Small updates
* Edited Errata
* Changed VReg resistor from 20k to 20.5k
* Changed ceramic cap symbols incorrectly listed as polarized
Parts:
- R56: value 20.0K -> 20.5K
Changed lines of the file:
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@@
       (effects (font (size 1.27 1.27)) (justify left))
     )
-    (property "Value" "20.0K" (at 200.66 45.7199 0)
+    (property "Value" "20.5K" (at 200.66 45.7199 0)
       (effects (font (size 1.27 1.27)) (justify left))
     )
@@
       (effects (font (size 1.27 1.27)) hide)
     )
-    (property "Datasheet" "https://www.mouser.com/ProductDetail/603-RC0603FR-103K3L" (at 198.12 44.45 0)
+    (property "Datasheet" "https://www.mouser.com/ProductDetail/YAGEO/RT0603FRE0720K5L" (at 198.12 44.45 0)
       (effects (font (size 1.27 1.27)) hide)
     )
