File: Harrison145_Main_Rev2/pitch_osc.kicad_sch (KiCad schematic)
At the start: 30 parts, among them Q1 MMBT3906, Q2 MMBT3906, Q3 SMP5484

Commit message: Small updates
* Edited Errata
* Changed VReg resistor from 20k to 20.5k
* Changed ceramic cap symbols incorrectly listed as polarized
Parts:
- C3: symbol Device:C_Polarized_Small_US -> Device:C_Small
Changed lines of the file:
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@@
     )
   )
-  (symbol (lib_id "Device:C_Polarized_Small_US") (at 98.425 90.17 0) (unit 1)
+  (symbol (lib_id "Device:C_Small") (at 98.425 90.17 0) (unit 1)
     (in_bom yes) (on_board yes) (dnp no) (fields_autoplaced)
-    (property "Reference" "C3" (at 100.965 88.4681 0)
+    (property "Reference" "C3" (at 101.6 89.5413 0)
       (effects (font (size 1.27 1.27)) (justify left))
     )
-    (property "Value" "100pF" (at 100.965 91.0081 0)
+    (property "Value" "100pF" (at 101.6 92.0813 0)
       (effects (font (size 1.27 1.27)) (justify left))
     )

Commit message: Progress on bringup of simulations in KiCAD 6 and KiCAD 7
Parts:
- added Vsim1: 7.5, symbol Simulation_SPICE:VDC
- C2: value 1uF -> 1u
- C3: value 100pF -> 100p
- C7: value 3.5-40pF -> 3.5pF
- CR1, CR2: value SM4001 -> temp=0
- L1: value 1mH -> 1m
- R48: value 100K -> 100k
- RV2: value 10K -> 10k
Connections:
- net GND: now also Vsim1.2
- net +7.5V renamed vsim
- net vsim: now also Vsim1.1; no longer R48.1, TP8.1
- new net: R48.1, TP8.1

Commit message: Remove kicad sims
Parts:
- removed Vsim1: 7.5, symbol Simulation_SPICE:VDC
Connections:
- net vsim is gone; now on net +7.5V: C1.1, Q3.2 (D), R1.1, R2.2, R5.1
- net +7.5V: now reaches R48.1, TP8.1
Changed lines of the file:
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@@
   (junction (at 65.405 93.345) (diameter 0) (color 0 0 0 0)
   )
+  (junction (at 57.785 76.835) (diameter 0) (color 0 0 0 0)
+  )
   (junction (at 98.425 93.345) (diameter 0) (color 0 0 0 0)
   )
@@
   (junction (at 172.72 91.44) (diameter 0) (color 0 0 0 0)
   )
-  (junction (at 57.785 101.5746) (diameter 0) (color 0 0 0 0)
-  )
   (junction (at 106.68 62.23) (diameter 0) (color 0 0 0 0)
   )
@@
     (stroke (width 0) (type default))
   )
-  (wire (pts (xy 33.02 80.3402) (xy 33.02 81.28))
+  (wire (pts (xy 57.785 74.93) (xy 57.785 76.835))
     (stroke (width 0) (type default))
   )
@@
     (stroke (width 0) (type default))
   )
-  (wire (pts (xy 57.785 101.5746) (xy 57.785 101.6))
-    (stroke (width 0) (type default))
-  )
   (wire (pts (xy 57.785 101.6) (xy 65.405 101.6))
     (stroke (width 0) (type default))
@@
     (stroke (width 0) (type default))
   )
-  (wire (pts (xy 33.02 101.5746) (xy 57.785 101.5746))
-    (stroke (width 0) (type default))
-  )
   (wire (pts (xy 107.315 101.6) (xy 115.57 101.6))
     (stroke (width 0) (type default))
@@
     (stroke (width 0) (type default))
   )
-  (wire (pts (xy 33.02 91.44) (xy 33.02 101.5746))
-    (stroke (width 0) (type default))
-  )
   (wire (pts (xy 106.68 62.23) (xy 95.25 62.23))
     (stroke (width 0) (type default))
@@
     (stroke (width 0) (type default))
   )
-  (wire (pts (xy 57.785 97.155) (xy 57.785 101.5746))
-    (stroke (width 0) (type default))
-  )
-  (label "vsim" (at 33.02 80.3402 90) (fields_autoplaced)
-    (effects (font (size 1.27 1.27)) (justify left bottom))
-  )
-  (label "vsim" (at 118.11 44.45 90) (fields_autoplaced)
-    (effects (font (size 1.27 1.27)) (justify left bottom))
+  (wire (pts (xy 57.785 97.155) (xy 57.785 101.6))
+    (stroke (width 0) (type default))
   )
   (label "FPO_OUT" (at 175.26 91.44 0) (fields_autoplaced)
-    (effects (font (size 1.27 1.27)) (justify left bottom))
-  )
-  (label "vsim" (at 172.72 70.485 90) (fields_autoplaced)
     (effects (font (size 1.27 1.27)) (justify left bottom))
   )
@@
     )
   )
+  (symbol (lib_id "power:+7.5V") (at 57.785 74.93 0) (unit 1)
+    (in_bom yes) (on_board yes) (dnp no)
+    (property "Reference" "#PWR0119" (at 57.785 78.74 0)
+      (effects (font (size 1.27 1.27)) hide)
+    )
+    (property "Value" "+7.5V" (at 57.785 69.85 0)
+      (effects (font (size 1.27 1.27)))
+    )
+    (property "Footprint" "" (at 57.785 74.93 0)
+      (effects (font (size 1.27 1.27)) hide)
+    )
+    (property "Datasheet" "" (at 57.785 74.93 0)
+      (effects (font (size 1.27 1.27)) hide)
+    )
+    (pin "1")
+    (instances
+      (project "Harrison145"
+        (path "/fe6a253a-fbe7-4763-8fb6-20765e8d5d9d/da22cfe7-cfea-4d69-bb2d-a68f4694277e"
+          (reference "#PWR0119") (unit 1)
+        )
+        (path "/fe6a253a-fbe7-4763-8fb6-20765e8d5d9d/dfa32f1a-941f-409e-ac16-27ee96c14cd3"
+          (reference "#PWR0129") (unit 1)
+        )
+      )
+    )
+  )
   (symbol (lib_id "Device:C_Small") (at 143.51 69.85 0) (unit 1)
     (in_bom yes) (on_board yes) (dnp no) (fields_autoplaced)
@@
     )
   )
-  (symbol (lib_id "Simulation_SPICE:VDC") (at 33.02 86.36 0) (unit 1)
-    (in_bom no) (on_board no) (dnp no) (fields_autoplaced)
-    (property "Reference" "Vsim1" (at 36.83 85.6892 0)
-      (effects (font (size 1.27 1.27)) (justify left))
-    )
-    (property "Value" "7.5" (at 36.83 88.2292 0)
-      (effects (font (size 1.27 1.27)) (justify left))
-    )
-    (property "Footprint" "" (at 33.02 86.36 0)
-      (effects (font (size 1.27 1.27)) hide)
-    )
-    (property "Datasheet" "~" (at 33.02 86.36 0)
-      (effects (font (size 1.27 1.27)) hide)
-    )
-    (property "Sim.Pins" "1=+ 2=-" (at 33.02 86.36 0)
-      (effects (font (size 0 0)) hide)
-    )
-    (property "Sim.Type" "DC" (at 33.02 86.36 0)
-      (effects (font (size 0 0)) hide)
-    )
-    (property "Sim.Device" "V" (at 33.02 86.36 0)
-      (effects (font (size 1.27 1.27)) (justify left) hide)
-    )
-    (property "Sim.Params" "ac=0 ph=0" (at 33.02 86.36 0)
-      (effects (font (size 1.27 1.27)) hide)
-    )
-    (pin "1")
-    (pin "2")
-    (instances
-      (project "Harrison145"
-        (path "/fe6a253a-fbe7-4763-8fb6-20765e8d5d9d/dfa32f1a-941f-409e-ac16-27ee96c14cd3"
-          (reference "Vsim1") (unit 1)
+  (symbol (lib_id "power:+7.5V") (at 172.72 70.485 0) (unit 1)
+    (in_bom yes) (on_board yes) (dnp no)
+    (property "Reference" "#PWR0119" (at 172.72 74.295 0)
+      (effects (font (size 1.27 1.27)) hide)
+    )
+    (property "Value" "+7.5V" (at 172.72 65.405 0)
+      (effects (font (size 1.27 1.27)))
+    )
+    (property "Footprint" "" (at 172.72 70.485 0)
+      (effects (font (size 1.27 1.27)) hide)
+    )
+    (property "Datasheet" "" (at 172.72 70.485 0)
+      (effects (font (size 1.27 1.27)) hide)
+    )
+    (pin "1")
+    (instances
+      (project "Harrison145"
+        (path "/fe6a253a-fbe7-4763-8fb6-20765e8d5d9d/da22cfe7-cfea-4d69-bb2d-a68f4694277e"
+          (reference "#PWR0119") (unit 1)
+        )
+        (path "/fe6a253a-fbe7-4763-8fb6-20765e8d5d9d/dfa32f1a-941f-409e-ac16-27ee96c14cd3"
+          (reference "#PWR0133") (unit 1)
         )
       )
@@
         )
       )
+    )
+  )
+  (symbol (lib_id "power:+7.5V") (at 118.11 44.45 0) (unit 1)
+    (in_bom yes) (on_board yes) (dnp no)
+    (property "Reference" "#PWR0119" (at 118.11 48.26 0)
+      (effects (font (size 1.27 1.27)) hide)
+    )
+    (property "Value" "+7.5V" (at 118.11 39.37 0)
+      (effects (font (size 1.27 1.27)))
+    )
+    (property "Footprint" "" (at 118.11 44.45 0)
+      (effects (font (size 1.27 1.27)) hide)
+    )
+    (property "Datasheet" "" (at 118.11 44.45 0)
+      (effects (font (size 1.27 1.27)) hide)
+    )
+    (pin "1")
+    (instances
+      (project "Harrison145"
+        (path "/fe6a253a-fbe7-4763-8fb6-20765e8d5d9d/da22cfe7-cfea-4d69-bb2d-a68f4694277e"
+          (reference "#PWR0119") (unit 1)
+        )
+        (path "/fe6a253a-fbe7-4763-8fb6-20765e8d5d9d/dfa32f1a-941f-409e-ac16-27ee96c14cd3"
+          (reference "#PWR0138") (unit 1)
+        )
+      )
