File: Harrison145_Main/AudioAmpVreg.kicad_sch (KiCad schematic)
At the start: 37 parts, among them J3 GROUND POINT, J4 LINE OUT, J5 9V IN, Q14 MMBT3904, Q15 MMBT3904, Q16 MMBT3906, U1 LDK320-ADJ_SOT23_SOT353

Commit message: Progress on bringup of simulations in KiCAD 6 and KiCAD 7
Parts:
- C32, C33, C35, C36, C37, C38, C39, C40, C41, CR6, D1, J3, J4, J5, JP5, Q14, Q15, Q16, R42, R43, R44, R45, R46, R47, R49, R50, R51, R52, R53, R54, R55, R56, R57, R58, TP5, TP7: Spice_Netlist_Enabled (none) -> N
Changed lines of the file:
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@@
       (effects (font (size 1.27 1.27)) (justify left) hide)
+    )
+    (property "Spice_Netlist_Enabled" "N" (id 4) (at 160.02 133.35 0)
+      (effects (font (size 1.27 1.27)) hide)
     )
     (pin "1")
@@
       (effects (font (size 1.27 1.27)) hide)
     )
+    (property "Spice_Netlist_Enabled" "N" (id 4) (at 161.29 45.72 0)
+      (effects (font (size 1.27 1.27)) hide)
+    )
     (pin "1")
     (pin "2")
@@
     )
     (property "Datasheet" "~" (id 3) (at 198.12 142.24 0)
+      (effects (font (size 1.27 1.27)) hide)
+    )
+    (property "Spice_Netlist_Enabled" "N" (id 4) (at 198.12 142.24 0)
       (effects (font (size 1.27 1.27)) hide)
     )
@@
       (effects (font (size 1.27 1.27)) hide)
     )
+    (property "Spice_Netlist_Enabled" "N" (id 4) (at 179.07 137.16 0)
+      (effects (font (size 1.27 1.27)) hide)
+    )
     (pin "1")
     (pin "2")
@@
       (effects (font (size 1.27 1.27)) hide)
     )
+    (property "Spice_Netlist_Enabled" "N" (id 4) (at 124.46 128.27 0)
+      (effects (font (size 1.27 1.27)) hide)
+    )
     (pin "1")
     (pin "2")
@@
       (effects (font (size 1.27 1.27)) hide)
     )
+    (property "Spice_Netlist_Enabled" "N" (id 4) (at 148.59 100.33 0)
+      (effects (font (size 1.27 1.27)) hide)
+    )
     (pin "1")
     (pin "2")
@@
     )
     (property "Datasheet" "https://www.mouser.com/ProductDetail/603-RC0603FR-07100KL" (id 3) (at 88.9 107.95 0)
+      (effects (font (size 1.27 1.27)) hide)
+    )
+    (property "Spice_Netlist_Enabled" "N" (id 4) (at 88.9 107.95 0)
       (effects (font (size 1.27 1.27)) hide)
     )
@@
       (effects (font (size 1.27 1.27)) hide)
     )
+    (property "Spice_Netlist_Enabled" "N" (id 4) (at 97.79 104.14 0)
+      (effects (font (size 1.27 1.27)) hide)
+    )
     (pin "1")
     (pin "2")
@@
       (effects (font (size 1.27 1.27)) hide)
     )
+    (property "Spice_Netlist_Enabled" "N" (id 4) (at 115.57 134.62 0)
+      (effects (font (size 1.27 1.27)) hide)
+    )
     (pin "1")
     (pin "2")
@@
       (effects (font (size 1.27 1.27)) hide)
     )
+    (property "Spice_Netlist_Enabled" "N" (id 4) (at 82.55 133.35 0)
+      (effects (font (size 1.27 1.27)) hide)
+    )
     (pin "1")
     (pin "2")
@@
     )
     (property "Datasheet" "https://www.mouser.com/ProductDetail/603-RC0603FR-13220RL" (id 3) (at 105.41 133.35 0)
+      (effects (font (size 1.27 1.27)) hide)
+    )
+    (property "Spice_Netlist_Enabled" "N" (id 4) (at 105.41 133.35 0)
       (effects (font (size 1.27 1.27)) hide)
     )
@@
       (effects (font (size 1.27 1.27)) hide)
     )
+    (property "Spice_Netlist_Enabled" "N" (id 4) (at 226.06 50.8 0)
+      (effects (font (size 1.27 1.27)) hide)
+    )
     (pin "1")
     (pin "2")
@@
       (effects (font (size 1.27 1.27)) hide)
     )
+    (property "Spice_Netlist_Enabled" "N" (id 4) (at 147.32 50.8 0)
+      (effects (font (size 1.27 1.27)) hide)
+    )
     (pin "1")
     (pin "2")
@@
       (effects (font (size 1.27 1.27)) hide)
     )
+    (property "Spice_Netlist_Enabled" "N" (id 4) (at 134.62 128.27 0)
+      (effects (font (size 1.27 1.27)) hide)
+    )
     (pin "1")
     (pin "2")
@@
     )
     (property "Datasheet" "~" (id 3) (at 237.49 62.23 0)
+      (effects (font (size 1.27 1.27)) hide)
+    )
+    (property "Spice_Netlist_Enabled" "N" (id 4) (at 237.49 62.23 0)
       (effects (font (size 1.27 1.27)) hide)
     )
@@
       (effects (font (size 1.27 1.27)) hide)
     )
+    (property "Spice_Netlist_Enabled" "N" (id 4) (at 148.59 138.43 0)
+      (effects (font (size 1.27 1.27)) hide)
+    )
     (pin "1")
     (pin "2")
@@
       (effects (font (size 1.27 1.27)) hide)
     )
+    (property "Spice_Netlist_Enabled" "N" (id 4) (at 162.56 124.46 0)
+      (effects (font (size 1.27 1.27)) hide)
+    )
     (pin "1")
     (pin "2")
@@
       (effects (font (size 1.27 1.27)) hide)
     )
+    (property "Spice_Netlist_Enabled" "N" (id 4) (at 76.2 116.84 0)
+      (effects (font (size 1.27 1.27)) hide)
+    )
     (pin "1")
     (pin "2")
@@
       (effects (font (size 1.27 1.27)) hide)
     )
+    (property "Spice_Netlist_Enabled" "N" (id 4) (at 161.29 55.88 0)
+      (effects (font (size 1.27 1.27)) hide)
+    )
     (pin "1")
     (pin "2")
@@
       (effects (font (size 1.27 1.27)) hide)
     )
+    (property "Spice_Netlist_Enabled" "N" (id 4) (at 212.09 50.8 0)
+      (effects (font (size 1.27 1.27)) hide)
+    )
     (pin "1")
     (pin "2")
@@
       (effects (font (size 1.27 1.27)) hide)
     )
+    (property "Spice_Netlist_Enabled" "N" (id 4) (at 129.54 134.62 0)
+      (effects (font (size 1.27 1.27)) hide)
+    )
     (pin "1")
     (pin "2")
@@
       (effects (font (size 1.27 1.27)) hide)
     )
+    (property "Spice_Netlist_Enabled" "N" (id 4) (at 114.3 39.37 0)
+      (effects (font (size 1.27 1.27)) hide)
+    )
     (pin "1")
   )
@@
       (effects (font (size 1.27 1.27)) hide)
     )
+    (property "Spice_Netlist_Enabled" "N" (id 4) (at 93.98 137.16 0)
+      (effects (font (size 1.27 1.27)) hide)
+    )
     (pin "1")
     (pin "2")
@@
       (effects (font (size 1.27 1.27)) hide)
     )
+    (property "Spice_Netlist_Enabled" "N" (id 4) (at 198.12 44.45 0)
+      (effects (font (size 1.27 1.27)) hide)
+    )
     (pin "1")
     (pin "2")
@@
     )
     (property "Datasheet" "https://www.mouser.com/ProductDetail/74-TMCP1E105KTRF" (id 3) (at 134.62 50.8 0)
+      (effects (font (size 1.27 1.27)) hide)
+    )
+    (property "Spice_Netlist_Enabled" "N" (id 4) (at 134.62 50.8 0)
       (effects (font (size 1.27 1.27)) hide)
     )
@@
       (effects (font (size 1.27 1.27)) hide)
     )
+    (property "Spice_Netlist_Enabled" "N" (id 4) (at 115.57 104.14 0)
+      (effects (font (size 1.27 1.27)) hide)
+    )
     (pin "1")
   )
@@
       (effects (font (size 1.27 1.27)) (justify left) hide)
     )
+    (property "Spice_Netlist_Enabled" "N" (id 4) (at 95.25 116.84 0)
+      (effects (font (size 1.27 1.27)) hide)
+    )
     (pin "1")
     (pin "2")
@@
     )
     (property "Datasheet" "https://www.mouser.com/ProductDetail/603-RC0603FR-073K92L" (id 3) (at 198.12 57.15 0)
+      (effects (font (size 1.27 1.27)) hide)
+    )
+    (property "Spice_Netlist_Enabled" "N" (id 4) (at 198.12 57.15 0)
       (effects (font (size 1.27 1.27)) hide)
     )
@@
       (effects (font (size 1.27 1.27)) hide)
     )
+    (property "Spice_Netlist_Enabled" "N" (id 4) (at 67.31 116.84 0)
+      (effects (font (size 1.27 1.27)) hide)
+    )
     (pin "1")
     (pin "2")
@@
       (effects (font (size 1.27 1.27)) (justify left) hide)
     )
+    (property "Spice_Netlist_Enabled" "N" (id 4) (at 160.02 105.41 0)
+      (effects (font (size 1.27 1.27)) hide)
+    )
     (pin "1")
     (pin "2")
@@
       (effects (font (size 1.27 1.27)) hide)
     )
+    (property "Spice_Netlist_Enabled" "N" (id 4) (at 191.77 142.24 0)
+      (effects (font (size 1.27 1.27)) hide)
+    )
     (pin "1")
   )
@@
       (effects (font (size 1.27 1.27)) hide)
     )
+    (property "Spice_Netlist_Enabled" "N" (id 4) (at 148.59 124.46 0)
+      (effects (font (size 1.27 1.27)) hide)
+    )
     (pin "1")
     (pin "2")
@@
       (effects (font (size 1.27 1.27)) hide)
     )
+    (property "Spice_Netlist_Enabled" "N" (id 4) (at 162.56 114.3 0)
+      (effects (font (size 1.27 1.27)) hide)
+    )
     (pin "1")
     (pin "2")
@@
       (effects (font (size 1.27 1.27)) hide)
     )
+    (property "Spice_Netlist_Enabled" "N" (id 4) (at 148.59 110.49 0)
+      (effects (font (size 1.27 1.27)) hide)
+    )
     (pin "1")
     (pin "2")
@@
       (effects (font (size 1.27 1.27)) hide)
     )
+    (property "Spice_Netlist_Enabled" "N" (id 4) (at 93.98 129.54 0)
+      (effects (font (size 1.27 1.27)) hide)
+    )
     (pin "1")
     (pin "2")
@@
       (effects (font (size 1.27 1.27)) hide)
     )
+    (property "Spice_Netlist_Enabled" "N" (id 4) (at 179.07 125.73 0)
+      (effects (font (size 1.27 1.27)) hide)
+    )
