File: Harrison145_Main/VolOsc.kicad_sch (KiCad schematic)
At the start: 29 parts, among them Q10 SMP5484, Q11 MMBT3906, Q12 MMBT3906

Commit message: Progress on bringup of simulations in KiCAD 6 and KiCAD 7
Parts:
- C25, C26, C27, C28, C29, C30, C31, CR4, CR5, JP4, L4, Q10, Q11, Q12, R31, R32, R33, R34, R35, R36, R37, R38, R39, R40, TP1, TP2, TP3, TP4: Spice_Netlist_Enabled (none) -> N
- RV1: Spice_Model (none) -> 10k; Spice_Netlist_Enabled (none) -> Y; Spice_Primitive (none) -> R
Changed lines of the file:
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@@
+      (effects (font (size 1.27 1.27)) hide)
+    )
+    (property "Spice_Model" "10k" (id 4) (at 100.965 127.635 0)
+      (effects (font (size 1.27 1.27)) hide)
+    )
+    (property "Spice_Netlist_Enabled" "Y" (id 5) (at 100.965 127.635 0)
+      (effects (font (size 1.27 1.27)) hide)
+    )
+    (property "Spice_Primitive" "R" (id 6) (at 100.965 127.635 0)
       (effects (font (size 1.27 1.27)) hide)
     )
@@
       (effects (font (size 1.27 1.27)) hide)
     )
+    (property "Spice_Netlist_Enabled" "N" (id 4) (at 172.72 127.635 0)
+      (effects (font (size 1.27 1.27)) hide)
+    )
     (pin "1")
     (pin "2")
@@
       (effects (font (size 1.27 1.27)) hide)
     )
+    (property "Spice_Netlist_Enabled" "N" (id 4) (at 204.47 113.03 0)
+      (effects (font (size 1.27 1.27)) hide)
+    )
     (pin "1")
     (pin "2")
@@
       (effects (font (size 1.27 1.27)) hide)
     )
+    (property "Spice_Netlist_Enabled" "N" (id 4) (at 141.605 131.445 0)
+      (effects (font (size 1.27 1.27)) hide)
+    )
     (pin "1")
     (pin "2")
@@
     )
     (property "Datasheet" "https://www.mouser.com/ProductDetail/74-TMCP1E105KTRF" (id 3) (at 108.585 132.08 0)
+      (effects (font (size 1.27 1.27)) hide)
+    )
+    (property "Spice_Netlist_Enabled" "N" (id 4) (at 108.585 132.08 0)
       (effects (font (size 1.27 1.27)) hide)
     )
@@
       (effects (font (size 1.27 1.27)) hide)
     )
+    (property "Spice_Netlist_Enabled" "N" (id 4) (at 97.79 119.38 0)
+      (effects (font (size 1.27 1.27)) hide)
+    )
     (pin "1")
   )
@@
       (effects (font (size 1.27 1.27)) hide)
     )
+    (property "Spice_Netlist_Enabled" "N" (id 4) (at 100.965 112.395 0)
+      (effects (font (size 1.27 1.27)) hide)
+    )
     (pin "1")
     (pin "2")
@@
       (effects (font (size 1.27 1.27)) hide)
     )
+    (property "Spice_Netlist_Enabled" "N" (id 4) (at 215.9 130.81 0)
+      (effects (font (size 1.27 1.27)) hide)
+    )
     (pin "1")
     (pin "2")
@@
     )
     (property "Datasheet" "https://www.mouser.com/ProductDetail/603-RC0603FR-07100KL" (id 3) (at 186.69 78.74 0)
+      (effects (font (size 1.27 1.27)) hide)
+    )
+    (property "Spice_Netlist_Enabled" "N" (id 4) (at 186.69 78.74 0)
       (effects (font (size 1.27 1.27)) hide)
     )
@@
       (effects (font (size 1.27 1.27)) hide)
     )
+    (property "Spice_Netlist_Enabled" "N" (id 4) (at 213.36 118.745 0)
+      (effects (font (size 1.27 1.27)) hide)
+    )
     (pin "1")
     (pin "2")
@@
       (effects (font (size 1.27 1.27)) hide)
     )
+    (property "Spice_Netlist_Enabled" "N" (id 4) (at 186.69 104.14 0)
+      (effects (font (size 1.27 1.27)) hide)
+    )
     (pin "1")
     (pin "2")
@@
     )
     (property "Datasheet" "https://www.mouser.com/ProductDetail/598-MC18FD331J-TF" (id 3) (at 158.75 127.635 0)
+      (effects (font (size 1.27 1.27)) hide)
+    )
+    (property "Spice_Netlist_Enabled" "N" (id 4) (at 158.75 127.635 0)
       (effects (font (size 1.27 1.27)) hide)
     )
@@
       (effects (font (size 1.27 1.27)) hide)
     )
+    (property "Spice_Netlist_Enabled" "N" (id 4) (at 108.585 123.825 0)
+      (effects (font (size 1.27 1.27)) hide)
+    )
     (pin "1")
   )
@@
     )
     (property "Datasheet" "https://www.mouser.com/ProductDetail/80-C0603C101K8RAUTO" (id 3) (at 141.605 123.19 0)
+      (effects (font (size 1.27 1.27)) hide)
+    )
+    (property "Spice_Netlist_Enabled" "N" (id 4) (at 141.605 123.19 0)
       (effects (font (size 1.27 1.27)) hide)
     )
@@
       (effects (font (size 1.27 1.27)) hide)
     )
+    (property "Spice_Netlist_Enabled" "N" (id 4) (at 114.935 127.635 0)
+      (effects (font (size 1.27 1.27)) hide)
+    )
     (pin "1")
     (pin "2")
@@
       (effects (font (size 1.27 1.27)) (justify left) hide)
     )
+    (property "Spice_Netlist_Enabled" "N" (id 4) (at 176.53 96.52 0)
+      (effects (font (size 1.27 1.27)) hide)
+    )
     (pin "1")
     (pin "2")
@@
       (effects (font (size 1.27 1.27)) hide)
     )
+    (property "Spice_Netlist_Enabled" "N" (id 4) (at 121.285 123.19 0)
+      (effects (font (size 1.27 1.27)) hide)
+    )
     (pin "1")
     (pin "2")
@@
     )
     (property "Datasheet" "https://www.mouser.com/ProductDetail/603-RC0603FR-103K3L" (id 3) (at 138.43 88.9 0)
+      (effects (font (size 1.27 1.27)) hide)
+    )
+    (property "Spice_Netlist_Enabled" "N" (id 4) (at 138.43 88.9 0)
       (effects (font (size 1.27 1.27)) hide)
     )
@@
       (effects (font (size 1.27 1.27)) hide)
     )
+    (property "Spice_Netlist_Enabled" "N" (id 4) (at 97.79 135.89 0)
+      (effects (font (size 1.27 1.27)) hide)
+    )
     (pin "1")
   )
@@
       (effects (font (size 1.27 1.27)) hide)
     )
+    (property "Spice_Netlist_Enabled" "N" (id 4) (at 187.96 128.27 0)
+      (effects (font (size 1.27 1.27)) hide)
+    )
     (pin "1")
     (pin "2")
@@
     )
     (property "Datasheet" "https://www.mouser.com/ProductDetail/74-TMCP1E105KTRF" (id 3) (at 149.86 88.9 0)
+      (effects (font (size 1.27 1.27)) hide)
+    )
+    (property "Spice_Netlist_Enabled" "N" (id 4) (at 149.86 88.9 0)
       (effects (font (size 1.27 1.27)) hide)
     )
@@
       (effects (font (size 1.27 1.27)) hide)
     )
+    (property "Spice_Netlist_Enabled" "N" (id 4) (at 196.85 118.745 0)
+      (effects (font (size 1.27 1.27)) hide)
+    )
     (pin "1")
     (pin "2")
@@
     )
     (property "Datasheet" "https://www.mouser.com/ProductDetail/Keystone-Electronics/5002" (id 3) (at 221.615 127.635 0)
+      (effects (font (size 1.27 1.27)) hide)
+    )
+    (property "Spice_Netlist_Enabled" "N" (id 4) (at 226.695 127.635 0)
       (effects (font (size 1.27 1.27)) hide)
     )
@@
       (effects (font (size 1.27 1.27)) hide)
     )
+    (property "Spice_Netlist_Enabled" "N" (id 4) (at 241.3 125.73 0)
+      (effects (font (size 1.27 1.27)) hide)
+    )
     (pin "1")
     (pin "2")
@@
     )
     (property "Datasheet" "https://www.mouser.com/ProductDetail/637-SM4001" (id 3) (at 121.285 132.08 0)
+      (effects (font (size 1.27 1.27)) hide)
+    )
+    (property "Spice_Netlist_Enabled" "N" (id 4) (at 121.285 132.08 0)
       (effects (font (size 1.27 1.27)) hide)
     )
@@
       (effects (font (size 1.27 1.27)) hide)
     )
+    (property "Spice_Netlist_Enabled" "N" (id 4) (at 138.43 101.6 0)
+      (effects (font (size 1.27 1.27)) hide)
+    )
     (pin "1")
     (pin "2")
@@
       (effects (font (size 1.27 1.27)) hide)
     )
+    (property "Spice_Netlist_Enabled" "N" (id 4) (at 161.29 85.09 0)
+      (effects (font (size 1.27 1.27)) hide)
+    )
     (pin "1")
     (pin "2")
@@
       (effects (font (size 1.27 1.27)) (justify left) hide)
     )
+    (property "Spice_Netlist_Enabled" "N" (id 4) (at 156.21 96.52 0)
+      (effects (font (size 1.27 1.27)) hide)
+    )
     (pin "1")
     (pin "2")
@@
       (effects (font (size 1.27 1.27)) hide)
     )
+    (property "Spice_Netlist_Enabled" "N" (id 4) (at 204.47 127 0)
+      (effects (font (size 1.27 1.27)) hide)
+    )
