File: Harrison145_Main/VolProcessor.kicad_sch (KiCad schematic)
At the start: 21 parts, among them J2 VOLUME ANTENNA, Q13 SMP5484, Q8 SMP5484, Q9 MMBT3904

Commit message: Progress on bringup of simulations in KiCAD 6 and KiCAD 7
Parts:
- C19, C20, C21, C22, C23, C24, C24_TEST1, C34, CR3, J2, L3, Q13, Q8, Q9, R26, R27, R28, R29, R30, R41, TP6: Spice_Netlist_Enabled (none) -> N
Changed lines of the file:
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@@
+      (effects (font (size 1.27 1.27)) hide)
+    )
+    (property "Spice_Netlist_Enabled" "N" (id 4) (at 191.77 86.36 0)
       (effects (font (size 1.27 1.27)) hide)
     )
@@
       (effects (font (size 1.27 1.27)) hide)
     )
+    (property "Spice_Netlist_Enabled" "N" (id 4) (at 124.46 97.79 0)
+      (effects (font (size 1.27 1.27)) hide)
+    )
     (pin "1")
     (pin "2")
@@
       (effects (font (size 1.27 1.27)) hide)
     )
+    (property "Spice_Netlist_Enabled" "N" (id 4) (at 143.51 91.44 0)
+      (effects (font (size 1.27 1.27)) hide)
+    )
     (pin "1")
     (pin "2")
@@
       (effects (font (size 1.27 1.27)) hide)
     )
+    (property "Spice_Netlist_Enabled" "N" (id 5) (at 63.5 109.22 0)
+      (effects (font (size 1.27 1.27)) hide)
+    )
     (pin "1")
     (pin "2")
@@
       (effects (font (size 1.27 1.27)) hide)
     )
+    (property "Spice_Netlist_Enabled" "N" (id 4) (at 179.07 97.79 0)
+      (effects (font (size 1.27 1.27)) hide)
+    )
     (pin "1")
     (pin "2")
@@
     )
     (property "Datasheet" "https://www.mouser.com/ProductDetail/603-RC0603FR-102K2L" (id 3) (at 158.75 114.3 0)
+      (effects (font (size 1.27 1.27)) hide)
+    )
+    (property "Spice_Netlist_Enabled" "N" (id 4) (at 158.75 114.3 0)
       (effects (font (size 1.27 1.27)) hide)
     )
@@
       (effects (font (size 1.27 1.27)) hide)
     )
+    (property "Spice_Netlist_Enabled" "N" (id 4) (at 80.01 109.22 0)
+      (effects (font (size 1.27 1.27)) hide)
+    )
     (pin "1")
     (pin "2")
@@
       (effects (font (size 1.27 1.27)) hide)
     )
+    (property "Spice_Netlist_Enabled" "N" (id 4) (at 167.64 109.22 0)
+      (effects (font (size 1.27 1.27)) hide)
+    )
     (pin "1")
     (pin "2")
@@
       (effects (font (size 1.27 1.27)) hide)
     )
+    (property "Spice_Netlist_Enabled" "N" (id 4) (at 176.53 116.84 0)
+      (effects (font (size 1.27 1.27)) hide)
+    )
     (pin "1")
     (pin "2")
@@
       (effects (font (size 1.27 1.27)) hide)
     )
+    (property "Spice_Netlist_Enabled" "N" (id 4) (at 209.55 105.41 0)
+      (effects (font (size 1.27 1.27)) hide)
+    )
     (pin "1")
     (pin "2")
@@
     )
     (property "Datasheet" "https://www.mouser.com/ProductDetail/106-SMP5484" (id 3) (at 218.44 91.44 0)
+      (effects (font (size 1.27 1.27)) hide)
+    )
+    (property "Spice_Netlist_Enabled" "N" (id 4) (at 218.44 91.44 0)
       (effects (font (size 1.27 1.27)) hide)
     )
@@
       (effects (font (size 1.27 1.27)) hide)
     )
+    (property "Spice_Netlist_Enabled" "N" (id 4) (at 201.93 82.55 0)
+      (effects (font (size 1.27 1.27)) hide)
+    )
     (pin "1")
   )
@@
       (effects (font (size 1.27 1.27)) hide)
     )
+    (property "Spice_Netlist_Enabled" "N" (id 4) (at 156.21 97.79 0)
+      (effects (font (size 1.27 1.27)) hide)
+    )
     (pin "1")
     (pin "2")
@@
       (effects (font (size 1.27 1.27)) hide)
     )
+    (property "Spice_Netlist_Enabled" "N" (id 4) (at 143.51 111.76 0)
+      (effects (font (size 1.27 1.27)) hide)
+    )
     (pin "1")
     (pin "2")
@@
     )
     (property "Datasheet" "https://www.mouser.com/ProductDetail/598-MC18FD331J-TF" (id 3) (at 91.44 109.22 0)
+      (effects (font (size 1.27 1.27)) hide)
+    )
+    (property "Spice_Netlist_Enabled" "N" (id 4) (at 91.44 109.22 0)
       (effects (font (size 1.27 1.27)) hide)
     )
@@
       (effects (font (size 1.27 1.27)) (justify left) hide)
     )
+    (property "Spice_Netlist_Enabled" "N" (id 4) (at 189.23 109.22 0)
+      (effects (font (size 1.27 1.27)) hide)
+    )
     (pin "1")
     (pin "2")
@@
     )
     (property "Datasheet" "https://www.mouser.com/ProductDetail/603-RC0603FR-102K2L" (id 3) (at 191.77 119.38 0)
+      (effects (font (size 1.27 1.27)) hide)
+    )
+    (property "Spice_Netlist_Enabled" "N" (id 4) (at 191.77 119.38 0)
       (effects (font (size 1.27 1.27)) hide)
     )
@@
       (effects (font (size 1.27 1.27)) hide)
     )
+    (property "Spice_Netlist_Enabled" "N" (id 4) (at 97.79 97.79 0)
+      (effects (font (size 1.27 1.27)) hide)
+    )
     (pin "1")
     (pin "2")
@@
     )
     (property "DNP" "1" (id 4) (at 105.41 109.22 0))
+    (property "Spice_Netlist_Enabled" "N" (id 5) (at 105.41 109.22 0)
+      (effects (font (size 1.27 1.27)) hide)
+    )
     (pin "1")
     (pin "2")
@@
       (effects (font (size 1.27 1.27)) hide)
     )
+    (property "Spice_Netlist_Enabled" "N" (id 4) (at 200.66 100.33 0)
+      (effects (font (size 1.27 1.27)) hide)
+    )
     (pin "1")
     (pin "2")
@@
       (effects (font (size 1.27 1.27)) hide)
     )
+    (property "Spice_Netlist_Enabled" "N" (id 4) (at 105.41 77.47 0)
+      (effects (font (size 1.27 1.27)) hide)
+    )
