File: Harrison145_Main/mixer.kicad_sch (KiCad schematic)
At the start: 17 parts, among them Q4 MMBT3904

Commit message: Progress on bringup of simulations in KiCAD 6 and KiCAD 7
Parts:
- C10, C11, C12, C13, C9, JP1, JP2, JP3, Q4, R11, R12, R13, R14, R15, R16, R17, R18: Spice_Netlist_Enabled (none) -> N
Changed lines of the file:
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@@
+      (effects (font (size 1.27 1.27)) hide)
+    )
+    (property "Spice_Netlist_Enabled" "N" (id 4) (at 135.89 113.03 0)
       (effects (font (size 1.27 1.27)) hide)
     )
@@
       (effects (font (size 1.27 1.27)) hide)
     )
+    (property "Spice_Netlist_Enabled" "N" (id 4) (at 125.73 113.03 0)
+      (effects (font (size 1.27 1.27)) hide)
+    )
     (pin "1")
     (pin "2")
@@
       (effects (font (size 1.27 1.27)) hide)
     )
+    (property "Spice_Netlist_Enabled" "N" (id 4) (at 199.39 91.44 0)
+      (effects (font (size 1.27 1.27)) hide)
+    )
     (pin "1")
     (pin "2")
@@
     )
     (property "Datasheet" "https://www.mouser.com/ProductDetail/603-RC0603FR-071KP" (id 3) (at 180.34 110.49 0)
+      (effects (font (size 1.27 1.27)) hide)
+    )
+    (property "Spice_Netlist_Enabled" "N" (id 4) (at 180.34 110.49 0)
       (effects (font (size 1.27 1.27)) hide)
     )
@@
       (effects (font (size 1.27 1.27)) hide)
     )
+    (property "Spice_Netlist_Enabled" "N" (id 4) (at 86.36 113.03 0)
+      (effects (font (size 1.27 1.27)) hide)
+    )
     (pin "1")
     (pin "2")
@@
       (effects (font (size 1.27 1.27)) hide)
     )
+    (property "Spice_Netlist_Enabled" "N" (id 4) (at 205.105 97.155 0)
+      (effects (font (size 1.27 1.27)) hide)
+    )
     (pin "1")
     (pin "2")
@@
       (effects (font (size 1.27 1.27)) (justify left) hide)
     )
+    (property "Spice_Netlist_Enabled" "N" (id 4) (at 168.275 97.79 0)
+      (effects (font (size 1.27 1.27)) hide)
+    )
     (pin "1")
     (pin "2")
@@
     )
     (property "Datasheet" "https://www.mouser.com/ProductDetail/603-RC0603FR-13150KL" (id 3) (at 159.385 86.36 0)
+      (effects (font (size 1.27 1.27)) hide)
+    )
+    (property "Spice_Netlist_Enabled" "N" (id 4) (at 159.385 86.36 0)
       (effects (font (size 1.27 1.27)) hide)
     )
@@
       (effects (font (size 1.27 1.27)) hide)
     )
+    (property "Spice_Netlist_Enabled" "N" (id 4) (at 144.78 113.03 0)
+      (effects (font (size 1.27 1.27)) hide)
+    )
     (pin "1")
     (pin "2")
@@
     )
     (property "Datasheet" "https://www.mouser.com/ProductDetail/603-RC0603FR-102K2L" (id 3) (at 170.815 85.725 0)
+      (effects (font (size 1.27 1.27)) hide)
+    )
+    (property "Spice_Netlist_Enabled" "N" (id 4) (at 170.815 85.725 0)
       (effects (font (size 1.27 1.27)) hide)
     )
@@
       (effects (font (size 1.27 1.27)) hide)
     )
+    (property "Spice_Netlist_Enabled" "N" (id 4) (at 111.125 113.03 0)
+      (effects (font (size 1.27 1.27)) hide)
+    )
     (pin "1")
     (pin "2")
@@
     )
     (property "Datasheet" "https://www.mouser.com/ProductDetail/603-RC0603FR-0710KL" (id 3) (at 99.06 113.03 0)
+      (effects (font (size 1.27 1.27)) hide)
+    )
+    (property "Spice_Netlist_Enabled" "N" (id 4) (at 99.06 113.03 0)
       (effects (font (size 1.27 1.27)) hide)
     )
@@
       (effects (font (size 1.27 1.27)) hide)
     )
+    (property "Spice_Netlist_Enabled" "N" (id 4) (at 220.98 91.44 0)
+      (effects (font (size 1.27 1.27)) hide)
+    )
     (pin "1")
     (pin "2")
@@
       (effects (font (size 1.27 1.27)) hide)
     )
+    (property "Spice_Netlist_Enabled" "N" (id 4) (at 170.815 114.3 0)
+      (effects (font (size 1.27 1.27)) hide)
+    )
     (pin "1")
     (pin "2")
@@
       (effects (font (size 1.27 1.27)) hide)
     )
+    (property "Spice_Netlist_Enabled" "N" (id 4) (at 180.34 118.11 0)
+      (effects (font (size 1.27 1.27)) hide)
+    )
     (pin "1")
     (pin "2")
@@
       (effects (font (size 1.27 1.27)) hide)
     )
+    (property "Spice_Netlist_Enabled" "N" (id 4) (at 159.385 110.49 0)
+      (effects (font (size 1.27 1.27)) hide)
+    )
     (pin "1")
     (pin "2")
@@
       (effects (font (size 1.27 1.27)) hide)
     )
+    (property "Spice_Netlist_Enabled" "N" (id 4) (at 193.04 97.155 0)
+      (effects (font (size 1.27 1.27)) hide)
+    )
