File: Harrison145_Main/pitch_osc.kicad_sch (KiCad schematic)
At the start: 28 parts, among them Q1 MMBT3906, Q2 MMBT3906, Q3 SMP5484

Commit message: Progress on bringup of simulations in KiCAD 6 and KiCAD 7
Parts:
- C1, C2: Spice_Model (none) -> 1u; Spice_Netlist_Enabled (none) -> Y; Spice_Primitive (none) -> C
- C3: Spice_Model (none) -> 100p; Spice_Netlist_Enabled (none) -> Y; Spice_Primitive (none) -> C
- C4, C5: Spice_Model (none) -> 10p; Spice_Netlist_Enabled (none) -> Y; Spice_Primitive (none) -> C
- C6: Spice_Model (none) -> 150p; Spice_Netlist_Enabled (none) -> Y; Spice_Primitive (none) -> C
- C7: value 3.5-40pF -> 3.5p; Range (none) -> 3.5-40pF; Spice_Model (none) -> 3.5p; Spice_Netlist_Enabled (none) -> Y; Spice_Primitive (none) -> C
- C8: Spice_Model (none) -> 0.01u; Spice_Netlist_Enabled (none) -> Y; Spice_Primitive (none) -> C
- CR1, CR2: Spice_Lib_File (none) -> Libraries\Diode.lib; Spice_Model (none) -> 1N4001; Spice_Netlist_Enabled (none) -> Y; Spice_Node_Sequence (none) -> 2 1; Spice_Primitive (none) -> D
- JP6, RV2: Spice_Netlist_Enabled (none) -> N
- L1: Spice_Model (none) -> 1m; Spice_Netlist_Enabled (none) -> Y; Spice_Primitive (none) -> L
- Q1, Q2: Spice_Lib_File (none) -> Libraries\BJT.lib; Spice_Model (none) -> MMBT3906; Spice_Netlist_Enabled (none) -> Y; Spice_Node_Sequence (none) -> 3 1 2; Spice_Primitive (none) -> Q
- Q3: Spice_Lib_File (none) -> Libraries\JFET.lib; Spice_Model (none) -> 2N5484; Spice_Netlist_Enabled (none) -> Y; Spice_Node_Sequence (none) -> 2 3 1; Spice_Primitive (none) -> J
- R1: Spice_Model (none) -> 3.3k; Spice_Netlist_Enabled (none) -> Y; Spice_Primitive (none) -> R
- R10, R8, R9: Spice_Model (none) -> 1M; Spice_Netlist_Enabled (none) -> Y; Spice_Primitive (none) -> R
- R2: Spice_Model (none) -> 22k; Spice_Netlist_Enabled (none) -> Y; Spice_Primitive (none) -> R
- R3: Spice_Model (none) -> 10k; Spice_Netlist_Enabled (none) -> Y; Spice_Primitive (none) -> R
- R4: Spice_Model (none) -> 100k; Spice_Netlist_Enabled (none) -> Y; Spice_Primitive (none) -> R
- R48: Spice_Model (none) -> 100k; Spice_Netlist_Enabled (none) -> Y
- R5: Spice_Model (none) -> 4.7M; Spice_Netlist_Enabled (none) -> Y; Spice_Primitive (none) -> R
- R6: Spice_Model (none) -> 2.7M; Spice_Netlist_Enabled (none) -> Y; Spice_Primitive (none) -> R
- R7: Spice_Model (none) -> 2.2k; Spice_Netlist_Enabled (none) -> Y; Spice_Primitive (none) -> R
